File: sequencer-io/leds.kicad_sch (KiCad schematic)
At the start: 34 parts

Commit message: edits
Parts:
- U12, U13, U14, U15, U16, U17, U18, U19: footprint SK6812MINI-E-012:SK6812MINI-E-012 -> SK6812MINI-E-012:SK6812MINI-E-012-ROT
Changed lines of the file:
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@@
 		(shape input)
 		(at 36.83 45.72 180)
-		(fields_autoplaced yes)
 		(effects
 			(font
@@
 			)
 		)
-		(property "Footprint" "SK6812MINI-E-012:SK6812MINI-E-012"
+		(property "Footprint" "SK6812MINI-E-012:SK6812MINI-E-012-ROT"
 			(at 156.21 78.74 0)
 			(effects
@@
 			)
 		)
-		(property "Footprint" "SK6812MINI-E-012:SK6812MINI-E-012"
+		(property "Footprint" "SK6812MINI-E-012:SK6812MINI-E-012-ROT"
 			(at 138.43 78.74 0)
 			(effects
@@
 			)
 		)
-		(property "Footprint" "SK6812MINI-E-012:SK6812MINI-E-012"
+		(property "Footprint" "SK6812MINI-E-012:SK6812MINI-E-012-ROT"
 			(at 193.04 78.74 0)
 			(effects
@@
 			)
 		)
-		(property "Footprint" "SK6812MINI-E-012:SK6812MINI-E-012"
+		(property "Footprint" "SK6812MINI-E-012:SK6812MINI-E-012-ROT"
 			(at 64.77 78.74 0)
 			(effects
@@
 			)
 		)
-		(property "Footprint" "SK6812MINI-E-012:SK6812MINI-E-012"
+		(property "Footprint" "SK6812MINI-E-012:SK6812MINI-E-012-ROT"
 			(at 82.55 78.74 0)
 			(effects
@@
 			)
 		)
-		(property "Footprint" "SK6812MINI-E-012:SK6812MINI-E-012"
+		(property "Footprint" "SK6812MINI-E-012:SK6812MINI-E-012-ROT"
 			(at 101.6 78.74 0)
 			(effects
@@
 			)
 		)
-		(property "Footprint" "SK6812MINI-E-012:SK6812MINI-E-012"
+		(property "Footprint" "SK6812MINI-E-012:SK6812MINI-E-012-ROT"
 			(at 175.26 78.74 0)
 			(effects
@@
 			)
 		)
-		(property "Footprint" "SK6812MINI-E-012:SK6812MINI-E-012"
+		(property "Footprint" "SK6812MINI-E-012:SK6812MINI-E-012-ROT"
 			(at 119.38 78.74 0)
 			(effects
