File: sequencer-io/ios.kicad_sch (KiCad schematic)
At the start: 48 parts, among them J1 ClockIn, J2 GateOut, J3 ClockOut, J4 PitchOut, J5 CVOut, J6 ResetIn, Q1 MMBT3904, Q2 MMBT3904, Q3 MMBT3906, Q4 MMBT3906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

Commit message: edits
Parts:
- removed R11, R12: 1k, Resistor_SMD:R_0603_1608Metric_Pad0.98x0.95mm_HandSolder, symbol Device:R_Small
Connections:
- net +5V: no longer R16.2, R9.2, RV1.1, RV2.1, RV3.1, RV4.1
- new net +3.3V: R16.2, R9.2, RV1.1, RV2.1, RV3.1, RV4.1
Other:
- moved on the sheet: C2, C3, SW24
