File: sequencer-io/sequencer-io.kicad_pcb (KiCad board)
At the start: 2 copper layers, 3.6 x 3.3 mm, 156 parts, among them IC1 TCA8418RTWR, J1 ClockIn, J2 GateOut, J3 ClockOut, J4 PitchOut, J5 CVOut, J6 ResetIn, J7 5V EXT, Q1 MMBT3904, Q2 MMBT3904, Q3 MMBT3906, Q4 MMBT3906, Q5 MMBT3906, Q7 DMG2305UX-7, SW1 SW_Push, SW10 SW_Push, SW11 SW_Push, SW12 SW_Push, SW13 SW_Push, SW14 SW_Push, SW15 SW_Push, SW16 SW_Push, SW17 SW_Push, SW18 SW_Push, SW19 SW_Push, SW2 SW_Push, SW20 SW_Push, SW21 SW_Push, SW22 SW_Push, SW23 SW_Push, SW24 RotaryEncoder, SW3 SW_Push, SW4 SW_Push, SW5 SW_Push, SW6 SW_Push, SW7 SW_Push, SW8 SW_Push, SW9 SW_Push, U1 74HC595, U20 SC0915, U21 MCP4822, U22 TL072

Commit message: edits
Parts:
- removed R11, R12: 1k, Resistor_SMD:R_0603_1608Metric_Pad0.98x0.95mm_HandSolder
- C1, C2, C22, C23, C24, C25, C3, Q3, Q4, Q5, R1, R2, R23, R24, R25, R28, R29, R3, R30, R31, R32, R33, R4, R5, R6, R7, R8, U1, U20, U21, U22: moved to B.Cu
- moved C3 226.9 mm to (35.0, 49.0), turned to 180 degrees
- moved C2 220.7 mm to (41.0, 49.0)
- moved SW24 212.9 mm to (38.1, 38.1)
- moved U1 190.7 mm to (97.0, 38.0)
- moved U2 183.5 mm to (76.2, 38.1)
- moved Q5 182.9 mm to (104.0, 28.0)
- moved R8 180.6 mm to (90.0, 27.0), turned to 180 degrees
- moved Q4 179.6 mm to (104.0, 36.0)
- moved R7 179.4 mm to (90.0, 30.0), turned to 180 degrees
- moved R6 178.3 mm to (90.0, 33.0), turned to 180 degrees
- moved R5 177.4 mm to (90.0, 36.0), turned to 180 degrees
- moved Q3 177.1 mm to (104.0, 44.0)
- moved R4 175.3 mm to (90.0, 39.0), turned to 180 degrees
- moved R3 174.2 mm to (90.0, 42.0), turned to 180 degrees
- moved R2 173.3 mm to (90.0, 45.0), turned to 180 degrees
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Connections:
- R16 pad 2: +5V -> +3.3V
- R9 pad 2: +5V -> +3.3V
- RV1 pad 1: +5V -> +3.3V
- RV2 pad 1: +5V -> +3.3V
- RV3 pad 1: +5V -> +3.3V
- RV4 pad 1: +5V -> +3.3V
- U20 pad 19: unconnected-(U20-GP14-Pad19) -> /IOs/ENC_B
- U20 pad 20: /LEDs/PXL -> /IOs/ENC_A
- U20 pad 24: unconnected-(U20-GP18-Pad24) -> /IOs/DIGIT_3
- U20 pad 25: unconnected-(U20-GP19-Pad25) -> /IOs/DIGIT_2
- U20 pad 26: unconnected-(U20-GP20-Pad26) -> /IOs/DIGIT_1
- U20 pad 34: unconnected-(U20-GP28-Pad34) -> /LEDs/PXL
Routing:
- net /IOs/ENC_B: track 0.00 -> 197.8 mm
- net /IOs/ENC_A: track 0.00 -> 192.8 mm
- net COL1: track 63.6 -> 201.0 mm, vias 0 -> 1
- net /IOs/DIGIT_1: track 0.00 -> 114.8 mm, vias 0 -> 2
- net /IOs/DIGIT_2: track 0.00 -> 104.4 mm, vias 0 -> 2
- net COL2: track 84.5 -> 179.1 mm, vias 1 -> 2
- net COL3: track 64.9 -> 159.3 mm, vias 1 -> 2
- net /IOs/DIGIT_3: track 0.00 -> 93.9 mm, vias 0 -> 2
- net COL0: track 136.6 -> 229.7 mm, vias 0 -> 1
- net /Switches/SDA: track 0.00 -> 87.0 mm, vias 0 -> 2
- net /Switches/SCL: track 0.00 -> 84.8 mm, vias 0 -> 2
- net +5V: track 1.72 -> 74.2 mm, vias 1 -> 20
- net Net-(U2-G): track 0.00 -> 58.6 mm
- net Net-(U2-DP): track 0.00 -> 51.2 mm
- net Net-(Q3-C): track 0.00 -> 42.5 mm, vias 0 -> 1
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- added copper zone on In2.Cu, net +3.3V
- added copper zone on In2.Cu, net +5V
- added copper zone on B.Cu, net GND
- added copper zone on F.Cu, net GND
- added copper zone on In1.Cu, net GND
Other:
- board size 3.6 x 3.3 mm -> 162 x 124 mm
- copper layers 2 -> 4
