File: sequencer-io/sequencer-io.kicad_sch (KiCad schematic)
At the start: 7 parts, among them J7 5V EXT, Q7 DMG2305UX-7, U20 SC0915

Commit message: removed rp2040
Parts:
- removed J7: 5V EXT, Connector_PinHeader_2.54mm:PinHeader_1x02_P2.54mm_Vertical, symbol Connector_Generic:Conn_01x02
- removed Q7: DMG2305UX-7, Package_TO_SOT_SMD:SOT-23, symbol Device:Q_PMOS_GSD
- removed U20: SC0915, SC0915:SC0915, symbol SC0915:SC0915
- added C1, C10, C11, C12, C13, C14, C15, C16, C17, C18, C19, C2, C20, C24, C3, C4, C5, C6, C7, C8, C9: 100nF, Capacitor_SMD:C_0603_1608Metric_Pad1.08x0.95mm_HandSolder, symbol Device:C_Small
- added C22, C23: 22pF, Capacitor_SMD:C_0603_1608Metric_Pad1.08x0.95mm_HandSolder, symbol Device:C_Small
- added D1, D10, D11, D12, D13, D14, D15, D16, D17, D18, D19, D2, D20, D21, D22, D23, D3, D4, D5, D6, D7, D8, D9: 1N4148W, Diode_SMD:D_SOD-323_HandSoldering, symbol Diode:1N4148W
- added D24, D27: 1SMB5918BT3G, Diode_SMD:D_SMB_Handsoldering, symbol Device:D_Zener_Small
- added D25: GATE, LED_THT:LED_D3.0mm_FlatTop, symbol Device:LED_Small
- added J1: GateOut, Connector_PinHeader_2.54mm:PinHeader_1x02_P2.54mm_Vertical, symbol Connector_Audio:AudioJack2
- added J2: ClockOut, Connector_PinHeader_2.54mm:PinHeader_1x02_P2.54mm_Vertical, symbol Connector_Audio:AudioJack2
- added J3: PitchOut, Connector_PinHeader_2.54mm:PinHeader_1x02_P2.54mm_Vertical, symbol Connector_Audio:AudioJack2
- added J4: CVOut, Connector_PinHeader_2.54mm:PinHeader_1x02_P2.54mm_Vertical, symbol Connector_Audio:AudioJack2
- added J5: ClockIn, Connector_PinHeader_2.54mm:PinHeader_1x02_P2.54mm_Vertical, symbol Connector_Audio:AudioJack2
- added J6: ResetIn, Connector_PinHeader_2.54mm:PinHeader_1x02_P2.54mm_Vertical, symbol Connector_Audio:AudioJack2
- added Q1, Q2, Q3: MMBT3906, Package_TO_SOT_SMD:SOT-23, symbol Transistor_BJT:MMBT3906
- added Q4, Q5: MMBT3904, Package_TO_SOT_SMD:SOT-23, symbol Transistor_BJT:MMBT3904
- added R1, R2, R22, R25, R3, R4: 1k, Resistor_SMD:R_0603_1608Metric_Pad0.98x0.95mm_HandSolder, symbol Device:R_Small
- added R10, R11, R12, R5, R6, R7, R8, R9: 100R, Resistor_SMD:R_0603_1608Metric_Pad0.98x0.95mm_HandSolder, symbol Device:R_Small
- added R13, R14, R15: 680R, Resistor_SMD:R_0603_1608Metric_Pad0.98x0.95mm_HandSolder, symbol Device:R_Small
- added R16, R23, R24, R26, R27: 10k, Resistor_SMD:R_0603_1608Metric_Pad0.98x0.95mm_HandSolder, symbol Device:R_Small
- added R17: 100k, Resistor_SMD:R_0603_1608Metric_Pad0.98x0.95mm_HandSolder, symbol Device:R_Small
- added R18, R21: 1M, Resistor_SMD:R_0603_1608Metric_Pad0.98x0.95mm_HandSolder, symbol Device:R_Small
- added RV1: PITCH, Connector_PinHeader_2.54mm:PinHeader_1x03_P2.54mm_Vertical, symbol Device:R_Potentiometer
- added RV2: OCTAVE, Connector_PinHeader_2.54mm:PinHeader_1x03_P2.54mm_Vertical, symbol Device:R_Potentiometer
- added RV3: LENGTH, Connector_PinHeader_2.54mm:PinHeader_1x03_P2.54mm_Vertical, symbol Device:R_Potentiometer
- added RV4: CV, Connector_PinHeader_2.54mm:PinHeader_1x03_P2.54mm_Vertical, symbol Device:R_Potentiometer
- added SW1, SW10, SW11, SW12, SW13, SW14, SW15, SW16, SW17, SW18, SW19, SW2, SW20, SW23, SW3, SW4, SW5, SW6, SW7, SW8, SW9: SW_Push, PCM_Switch_Keyboard_Cherry_MX:SW_Cherry_MX_PCB_1.00u, symbol Switch:SW_Push
- added SW21, SW22: SW_Push, PCM_Switch_Keyboard_Cherry_MX:SW_Cherry_MX_PCB_2.00u, symbol Switch:SW_Push
- added SW24: RotaryEncoder, EC12E2430404:EC12E2430404, symbol Device:RotaryEncoder
- added TP1, TP10, TP11, TP12, TP13, TP2, TP3, TP4, TP5, TP6, TP7, TP8, TP9: TestPoint, symbol Connector:TestPoint
- added U1: 74HC595, Package_SO:SOIC-16_3.9x9.9mm_P1.27mm, symbol 74xx:74HC595
- added U10, U11, U3, U4, U5, U6, U7, U8, U9: ~, SK6812MINI-E-012:SK6812MINI-E-012, symbol SK6812MINI-E-012:SK6812MINI-E-012
- added U12, U13, U14, U15, U16, U17, U18, U19: ~, SK6812MINI-E-012:SK6812MINI-E-012-ROT, symbol SK6812MINI-E-012:SK6812MINI-E-012
- added U2: ~, FJ5361BH:FJ5361BH, symbol FJ5361BH:FJ5361BH
- added U20: TL072, Package_SO:SOIC-8_3.9x4.9mm_P1.27mm, symbol Amplifier_Operational:TL072
- added U21: MCP4822, Package_SO:SOIC-8_3.9x4.9mm_P1.27mm, symbol Analog_DAC:MCP4822
- C21: value 47uF -> 100nF
- R20: value 10k -> 100k
Connections:
- net Switches/SDA is gone; now on net +3.3V: R19.2
- net +3.3V: now also R16.2, RV1.1, RV2.1, RV3.1, RV4.1; no longer R19.1, R20.1
- net +5V: now also C1.2, C10.2, C11.2, C12.2, C13.2, C14.2, C15.2, C16.2, C17.2, C18.2, C19.2, C20.2, C4.2, C5.2, C6.2, C7.2, C8.2, C9.2, Q1.2 (E), Q2.2 (E), Q3.2 (E), U1.10 (~{SRCLR}), U1.16 (VCC), U10.3 (VDD), U11.3 (VDD), U12.3 (VDD), U13.3 (VDD), U14.3 (VDD), U15.3 (VDD), U16.3 (VDD), U17.3 (VDD), U18.3 (VDD), U19.3 (VDD), U21.1 (Vdd), U3.3 (VDD), U4.3 (VDD), U5.3 (VDD), U6.3 (VDD), U7.3 (VDD), U8.3 (VDD), U9.3 (VDD); no longer D26.1 (K)
- net GND: now also D26.2 (A), C1.1, C10.1, C11.1, C12.1, C13.1, C14.1, C15.1, C16.1, C17.1, C18.1, C19.1, C2.1, C20.1, C3.1, C4.1, C5.1, C6.1, C7.1, C8.1, C9.1, D24.2 (A), D27.2 (A), J1.S, J2.S, J3.S, J4.S, J5.S, J6.S, Q4.2 (E), Q5.2 (E), R18.1, R2.1, R21.1, R23.1, R26.1, RV4.3, SW24.C, U1.13 (~{OE}), U1.8 (GND), U10.1 (GND), U11.1 (GND), U12.1 (GND), U13.1 (GND), U14.1 (GND), U15.1 (GND), U16.1 (GND), U17.1 (GND), U18.1 (GND), U19.1 (GND), U21.5 (~{LDAC}), U21.7 (Vss), U3.1 (GND), U4.1 (GND), U5.1 (GND), U6.1 (GND), U7.1 (GND), U8.1 (GND), U9.1 (GND)
- net Switches/SCL: no longer names the net of R20.2
- net Switches/SCL: now also Q5.1 (B), R21.2
- new net: D17.2 (A), SW17.2
- new net: Q3.1 (B), R15.1
- new net: D25.2 (A), D26.1 (K), R1.1, R3.1
- new net: D14.2 (A), SW14.2
- new net: D13.2 (A), SW13.2
- new net: R9.2, U2.1 (E)
- new net: R10.2, U2.10 (F)
- new net: R5.2, U2.11 (A)
- new net: Q1.3 (C), U2.12 (DIGIT_1)
- new net: R8.2, U2.2 (D)
- new net: R12.2, U2.3 (DP)
- new net: R7.2, U2.4 (C)
- new net: R11.2, U2.5 (G)
- new net: R6.2, U2.7 (B)
- new net: Q3.3 (C), U2.8 (DIGIT_3)
- new net: Q2.3 (C), U2.9 (DIGIT_2)
- new net: R6.1, U1.1 (QB)
- new net: U7.4 (DOUT), U8.2 (DIN)
- new net: U8.4 (DOUT), U9.2 (DIN)
- new net: J2.T, R4.1
- new net: D15.2 (A), SW15.2
- new net: D20.2 (A), SW20.2
- new net: D2.2 (A), SW2.2
- new net: R12.1, U1.7 (QH)
- new net: C23.2, R25.1, U20.7
- new net: U20.5 (+), U21.6 (VB)
- new net: U20.3 (+), U21.8 (VA)
- new net: J5.T, R17.1
- new net: C22.1, R23.2, R24.1, U20.2 (-)
- new net: C22.2, R22.1, U20.1
- new net: U18.4 (DOUT), U19.2 (DIN)
- new net: J1.T, R3.2
- new net: TP13.1, U3.2 (DIN)
- new net: U5.4 (DOUT), U6.2 (DIN)
- new net: U6.4 (DOUT), U7.2 (DIN)
- new net: D12.2 (A), SW12.2
- new net: D9.2 (A), SW9.2
- new net: D22.2 (A), SW22.2
- new net: U10.4 (DOUT), U11.2 (DIN)
- new net: U11.4 (DOUT), U12.2 (DIN)
- new net: D5.2 (A), SW5.2
- new net: C23.1, R26.2, R27.1, U20.6 (-)
- new net: D11.2 (A), SW11.2
- new net: D25.1 (K), R2.2
- new net: R8.1, U1.3 (QD)
- new net: R10.1, U1.5 (QF)
- new net: D16.2 (A), SW16.2
- new net: D18.2 (A), SW18.2
- new net: U4.4 (DOUT), U5.2 (DIN)
- new net: J6.T, R20.1
- new net: D4.2 (A), SW4.2
- new net: D8.2 (A), SW8.2
- new net: D7.2 (A), SW7.2
- new net: Q2.1 (B), R14.1
- new net: R7.1, U1.2 (QC)
- new net: R5.1, U1.15 (QA)
- new net: R9.1, U1.4 (QE)
- new net: R11.1, U1.6 (QG)
- new net: Q1.1 (B), R13.1
- new net: D23.2 (A), SW23.2
- new net: U3.4 (DOUT), U4.2 (DIN)
- new net: Q4.1 (B), R17.2, R18.2
- new net: D1.2 (A), SW1.2
- new net: D6.2 (A), SW6.2
- new net: U16.4 (DOUT), U17.2 (DIN)
- new net: U17.4 (DOUT), U18.2 (DIN)
- new net: D19.2 (A), SW19.2
- new net: D3.2 (A), SW3.2
- new net: D10.2 (A), SW10.2
- new net: U12.4 (DOUT), U13.2 (DIN)
- new net: U13.4 (DOUT), U14.2 (DIN)
- new net: U10.2 (DIN), U9.4 (DOUT)
- new net: U14.4 (DOUT), U15.2 (DIN)
- new net: U15.4 (DOUT), U16.2 (DIN)
- new net: D21.2 (A), SW21.2
- new net +12V: C24.2, U20.8 (V+)
- new net -12V: C24.1, U20.4 (V-)
- new net AD1: RV1.2
- new net AD2: RV2.2
- new net AD3: RV3.2
- new net AD4: RV4.2
- new net CLKIN: Q4.3 (C), R16.1
- new net CLKOUT: D27.1 (K), R4.2
- new net COL0: SW1.1, SW13.1, SW21.1, SW5.1, TP5.1
- new net COL1: SW14.1, SW2.1, SW22.1, SW6.1, TP6.1
- new net COL2: SW15.1, SW23.1, SW3.1, SW7.1, TP7.1
- new net COL3: SW16.1, SW4.1, SW8.1, TP8.1
- new net COL4: SW17.1, SW9.1, TP9.1
- new net COL5: SW10.1, SW18.1, TP10.1
- new net COL6: SW11.1, SW19.1, TP11.1
- new net COL7: SW12.1, SW20.1, TP12.1
- new net CS_DAC: U21.2 (~{CS})
- new net CS_SHIFT: U1.12 (RCLK)
- new net CV: J4.T, R25.2, R27.2
- new net DIGIT_1: R13.2
- new net DIGIT_2: R14.2
- new net DIGIT_3: R15.2
- new net ENC_A: C3.2, SW24.A
- new net ENC_B: C2.2, SW24.B
- new net GATE: D24.1 (K), R1.2
- new net MOSI: U21.4 (SDI)
- new net PITCH: J3.T, R22.2, R24.2
- new net ROW0: D1.1 (K), D2.1 (K), D3.1 (K), D4.1 (K), TP1.1
- new net ROW1: D10.1 (K), D11.1 (K), D12.1 (K), D5.1 (K), D6.1 (K), D7.1 (K), D8.1 (K), D9.1 (K), TP2.1
- new net ROW2: D13.1 (K), D14.1 (K), D15.1 (K), D16.1 (K), D17.1 (K), D18.1 (K), D19.1 (K), D20.1 (K), TP3.1
- new net ROW3: D21.1 (K), D22.1 (K), D23.1 (K), TP4.1
- new net RSTIN: Q5.3 (C), R19.1
- new net SCLK: U1.11 (SRCLK), U21.3 (SCK)
- new net SER: U1.14 (SER)
- no-connect marks 7 -> 1
Other:
- removed sheet DAC
- removed sheet IOs
- removed sheet LEDs
- removed sheet Switches
- note added: "7 SEGMENT DISPLAY"
- note added: "ADDRESSABLE LEDs"
- note added: "DAC"
- note added: "ENCODER"
- note added: "INPUT JACKS"
- note added: "LEDs DECOUPLING"
- note added: "OUTPUT JACKS"
- note added: "POTENTIOMETERS"
- note added: "SWITCH MATRIX"
