File: 16-steps/16-steps.kicad_pcb (KiCad board)
At the start: 2 copper layers, 164 x 95 mm, 91 parts, among them J1 COLs 0-3, J2 ROWs / LEDs, J3 COLs 4-7, SW1 SW_Push, SW10 SW_Push, SW11 SW_Push, SW12 SW_Push, SW13 SW_Push, SW14 SW_Push, SW15 SW_Push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

Commit message: tidy up - remove duplicates
Routing:
- net COL2: track 256.0 -> 257.4 mm
