File: hardware/16-steps/16-steps.kicad_sch (KiCad schematic)
At the start: 91 parts, among them J1 COLs 0-3, J2 ROWs / LEDs, J3 COLs 4-7, SW1 SW_Push, SW10 SW_Push, SW11 SW_Push, SW12 SW_Push, SW13 SW_Push, SW14 SW_Push, SW15 SW_Push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

Commit message: clean up, added pdf schematics
Other:
- title: (none) -> Cherry MX 16-step Sequencer
- moved on the sheet: H1, H2, H3, H4, H5, H6, H7, H8, J1, J2, J3
