File: hardware/jacks-n-dac/jacks-n-dac.kicad_sch (KiCad schematic)
At the start: 41 parts, among them J1 DAC, J10 ResetIn, J2 12V IN, J3 5V IN, J4 GateOut, J5 ClockIn, J6 ClockOut, J7 INPUTS, J8 PitchOut, J9 CVOut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

Commit message: clean up, added pdf schematics
Other:
- note added: "MISC"
- title: (none) -> DAC, Opamp and Jacks Board
- moved on the sheet: H1, H2, H3, J1, J2, J3, J7
