File: hardware/7-segment/7-segment.kicad_pcb (KiCad board)
At the start: 2 copper layers, 68.6 x 27.9 mm, 20 parts, among them J1 I/O, Q1 MMBT3906, Q2 MMBT3906, Q3 MMBT3906, U2 74HC595

Commit message: corrected resistor values
Parts:
- R10, R11, R4, R5, R6, R7, R8, R9: value 100R -> 220R
Changed lines of the file:
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@@
 			)
 		)
-		(property "Value" "100R"
+		(property "Value" "220R"
 			(at 0 1.43 90)
 			(layer "F.Fab")
@@
 			)
 		)
-		(property "Value" "100R"
+		(property "Value" "220R"
 			(at 0 1.43 90)
 			(layer "F.Fab")
@@
 			)
 		)
-		(property "Value" "100R"
+		(property "Value" "220R"
 			(at 0 1.43 90)
 			(layer "F.Fab")
@@
 			)
 		)
-		(property "Value" "100R"
+		(property "Value" "220R"
 			(at 0 1.43 90)
 			(layer "F.Fab")
@@
 			)
 		)
-		(property "Value" "100R"
+		(property "Value" "220R"
 			(at 0 1.43 90)
 			(layer "F.Fab")
@@
 			)
 		)
-		(property "Value" "100R"
+		(property "Value" "220R"
 			(at 0 1.43 90)
 			(layer "F.Fab")
@@
 			)
 		)
-		(property "Value" "100R"
+		(property "Value" "220R"
 			(at 0 1.43 90)
 			(layer "F.Fab")
@@
 			)
 		)
-		(property "Value" "100R"
+		(property "Value" "220R"
 			(at 0 1.43 90)
 			(layer "F.Fab")
