File: hardware/7-segment/7-segment.kicad_sch (KiCad schematic)
At the start: 20 parts, among them J1 I/O, Q1 MMBT3906, Q2 MMBT3906, Q3 MMBT3906, U2 74HC595

Commit message: clean up, added pdf schematics
Other:
- title: (none) -> 3 Digits 7 Segment Display 
- moved on the sheet: H1, H2, H3, J1, Q1, Q2, Q3, R1, R10, R11, R2, R3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

Commit message: corrected resistor values
Parts:
- R10, R11, R4, R5, R6, R7, R8, R9: value 100R -> 220R
Changed lines of the file:
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@@
 	(label "DIG1"
 		(at 92.71 76.2 180)
-		(fields_autoplaced yes)
 		(effects
 			(font
@@
 	(label "DIG3"
 		(at 140.97 55.88 180)
-		(fields_autoplaced yes)
 		(effects
 			(font
@@
 	(label "SER"
 		(at 213.36 73.66 0)
-		(fields_autoplaced yes)
 		(effects
 			(font
@@
 	(label "DIG1"
 		(at 213.36 60.96 0)
-		(fields_autoplaced yes)
 		(effects
 			(font
@@
 	(label "SRCLK"
 		(at 69.85 124.46 180)
-		(fields_autoplaced yes)
 		(effects
 			(font
@@
 	(label "RCLK"
 		(at 69.85 132.08 180)
-		(fields_autoplaced yes)
 		(effects
 			(font
@@
 	(label "SRCLK"
 		(at 213.36 68.58 0)
-		(fields_autoplaced yes)
 		(effects
 			(font
@@
 	(label "DIG2"
 		(at 213.36 63.5 0)
-		(fields_autoplaced yes)
 		(effects
 			(font
@@
 	(label "SER"
 		(at 69.85 119.38 180)
-		(fields_autoplaced yes)
 		(effects
 			(font
@@
 	(label "RCLK"
 		(at 213.36 71.12 0)
-		(fields_autoplaced yes)
 		(effects
 			(font
@@
 	(label "DIG3"
 		(at 213.36 66.04 0)
-		(fields_autoplaced yes)
 		(effects
 			(font
@@
 	(label "DIG2"
 		(at 116.84 66.04 180)
-		(fields_autoplaced yes)
 		(effects
 			(font
@@
 			)
 		)
-		(property "Value" "100R"
+		(property "Value" "220R"
 			(at 106.934 108.204 90)
 			(effects
@@
 			)
 		)
-		(property "Value" "100R"
+		(property "Value" "220R"
 			(at 99.314 108.204 90)
 			(effects
@@
 			)
 		)
-		(property "Value" "100R"
+		(property "Value" "220R"
 			(at 104.394 108.204 90)
 			(effects
@@
 			)
 		)
-		(property "Value" "100R"
+		(property "Value" "220R"
 			(at 101.854 108.204 90)
 			(effects
@@
 			)
 		)
-		(property "Value" "100R"
+		(property "Value" "220R"
 			(at 112.014 108.204 90)
 			(effects
@@
 			)
 		)
-		(property "Value" "100R"
+		(property "Value" "220R"
 			(at 109.474 108.204 90)
 			(effects
@@
 			)
 		)
-		(property "Value" "100R"
+		(property "Value" "220R"
 			(at 117.094 108.204 90)
 			(effects
@@
 			)
 		)
-		(property "Value" "100R"
+		(property "Value" "220R"
 			(at 114.554 108.204 90)
 			(effects
